Commit message: S

File: urdf/sweepee/sweepee.urdf.xacro (robot description, xacro)
@@ -1,22 +1,11 @@
 <?xml version="1.0"?>
-<robot name="eureca" xmlns:xacro="http://ros.org/wiki/xacro">
+<robot name="sweepee" xmlns:xacro="http://ros.org/wiki/xacro">
 <!--   <xacro:include filename="$(find eureca_description)/urdf/sweepee/sweepee.gazebo.xacro" /> -->
   <xacro:include filename="$(find ros2_assembly)/urdf/sweepee/sweepee.xacro" />
 <!-- common stuff -->
   <xacro:include filename="$(find ur_description)/urdf/common.gazebo.xacro" />
-  <!-- ur10 -->
-  <xacro:include filename="$(find ur_description)/urdf/ur10.urdf.xacro" />
   <xacro:property name="M_PI" value="3.14159"/>
   <xacro:sweepee robot_namespace="/" >
     <origin xyz="0 0 0" rpy="0 0 0" />
   </xacro:sweepee>
-  <!-- arm -->
-  <xacro:ur10_robot prefix="ur10_" joint_limited="false"
-    transmission_hw_interface="hardware_interface/PositionJointInterface"
-  />
-  <joint name="world_joint" type="fixed">
-    <parent link="base_footprint" />
-    <child link = "ur10_base_link" />
-    <origin xyz="0.0 0.0 0.30" rpy="0.0 0.0 0.0" />
-  </joint>
 </robot>

File: urdf/system.urdf.xacro (robot description, xacro)
@@ -7,4 +7,5 @@
   <!-- ur10 -->
   <xacro:include filename="$(find ur_description)/urdf/ur10.urdf.xacro" />
+  <xacro:include filename="$(find ros2_assembly)/urdf/components/fuselage.xacro"/>
   <xacro:property name="M_PI" value="3.14159"/>
   <xacro:sweepee robot_namespace="/" >
@@ -21,4 +22,8 @@
   </joint>
   <link name="world"/>
+  <joint name="world_sweepee" type="floating">
+    <parent link="world" />
+    <child link = "base_footprint" />
+  </joint>
   <xacro:include filename="$(find ur5_on_guide_description)/urdf/ur5_on_guide.urdf.xacro" />
   <xacro:ur5_on_guide/>
@@ -28,3 +33,6 @@
     <origin xyz="0 0 0.0" rpy="0 0 0" />
   </joint>
+  <xacro:fuselage link_name="fuselage" parent="world" model="fuselage_nopanelfixing" >
+      <origin xyz="-4.2672  0 0.095" rpy="0 0 0" />
+  </xacro:fuselage>
 </robot>

File: urdf/ur5.urdf.xacro (robot description, xacro)
@@ -1,4 +1,4 @@
 <?xml version="1.0"?>
-<robot name="eureca" xmlns:xacro="http://ros.org/wiki/xacro">
+<robot name="ur5" xmlns:xacro="http://ros.org/wiki/xacro">
   <link name="world"/>
   <xacro:include filename="$(find ur5_on_guide_description)/urdf/ur5_on_guide.urdf.xacro" />
